File: pcb/bebox_encoder.brd (EAGLE design)
At the start: 58.9 x 21.6 mm, 7 parts, among them IC1 2590, J1 SJ-435107RS, J6 SJ-435107RS, U1 GP1A57HR, U2 GP1A57HR

Commit message: Updated screenprints.
Other:
- board text added: "A. Sugden v1.0"
- board text added: "BeBox"
- board text added: "ENCODER"
Changed lines of the file:
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@@
 <?xml version="1.0" encoding="utf-8"?>
 <!DOCTYPE eagle SYSTEM "eagle.dtd">
-<eagle version="9.3.1">
+<eagle version="9.3.2">
 <drawing>
 <settings>
@@
 <text x="37.973" y="23.495" size="0.8128" layer="22" rot="MR0">BEAM BREAK</text>
 <text x="37.846" y="13.716" size="0.8128" layer="22" rot="MR0">BEAM BREAK</text>
+<text x="40.005" y="28.702" size="0.8128" layer="21">A. Sugden v1.0</text>
+<text x="11.938" y="27.305" size="1.6764" layer="21">BeBox</text>
+<text x="11.938" y="25.908" size="1.016" layer="21">ENCODER</text>
 </plain>
 <attributes>
