File: pcb/bebox_main_itsybitsy.brd (EAGLE design)
At the start: 92.9 x 35.6 mm, 30 parts, among them J1 SJ-435107RS, J2 SJ-435107RS, J4 SJ-435107RS, J6 PJ-102AH, P2 OSTTE020104, P3 OSTTE020104, P4 OSTTE020104, P5 OSTTE020104, Q1 2N7000, Q2 2N7000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

Commit message: Updated screenprints.
Connections:
- net N$3: now also R2.2
Routing:
- net N$3: track 41.9 -> 51.1 mm
Other:
- board text added: "5V POWER REGULATOR"
- board text removed: "ADAFRUIT ITSYBITSY M4"
Changed lines of the file:
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@@
 <layer number="23" name="tOrigins" color="15" fill="1" visible="yes" active="yes"/>
 <layer number="24" name="bOrigins" color="15" fill="1" visible="yes" active="yes"/>
-<layer number="25" name="tNames" color="7" fill="1" visible="no" active="yes"/>
+<layer number="25" name="tNames" color="7" fill="1" visible="yes" active="yes"/>
 <layer number="26" name="bNames" color="7" fill="1" visible="no" active="yes"/>
 <layer number="27" name="tValues" color="7" fill="1" visible="no" active="yes"/>
@@
 <text x="39.37" y="43.18" size="1.27" layer="21">SOL 2</text>
 <text x="52.07" y="43.18" size="1.27" layer="21">SOL 1</text>
-<text x="93.98" y="21.59" size="1.778" layer="21" rot="R90">ADAFRUIT
-ITSYBITSY M4</text>
 <text x="79.121" y="43.815" size="1.27" layer="21" rot="R180">4.7k</text>
 <text x="68.961" y="38.735" size="1.27" layer="21" rot="R180">4.7k</text>
+<text x="63.373" y="28.321" size="1.016" layer="25">5V POWER
+REGULATOR</text>
 </plain>
 <attributes>
@@
 <wire x1="86.35619375" y1="38.845525" x2="85.09" y2="37.57933125" width="0.4064" layer="1"/>
 <wire x1="86.35619375" y1="43.17619375" x2="86.35619375" y2="38.845525" width="0.4064" layer="1"/>
+<contactref element="R2" pad="2"/>
+<wire x1="77.47" y1="40.64" x2="81.28" y2="36.83" width="0.4064" layer="1"/>
+<wire x1="81.28" y1="36.83" x2="85.09" y2="36.83" width="0.4064" layer="1"/>
 </signal>
 </signals>
